File: eurorack-PSU-extension/eurorack-PSU-extension.kicad_sch (KiCad schematic)
At the start: 8 parts, among them J1 Screw_Terminal_01x03, J10 Screw_Terminal_01x03, J2 Conn_02x05_Top_Bottom, J3 Conn_02x05_Top_Bottom, J4 Conn_02x05_Top_Bottom, J5 Conn_02x05_Top_Bottom, J6 Conn_02x05_Top_Bottom, J7 Conn_02x05_Top_Bottom

Commit message: PSU extension rework
Parts:
- removed J6: Conn_02x05_Top_Bottom, Connector_IDC:IDC-Header_2x05_P2.54mm_Vertical, symbol Connector_Generic:Conn_02x05_Odd_Even
- added J3, J5, J9: Conn_02x05_Top_Bottom, Connector_IDC:IDC-Header_2x05_P2.54mm_Vertical, symbol Connector_Generic:Conn_02x05_Odd_Even
- J1, J10: footprint TerminalBlock:TerminalBlock_bornier-3_P5.08mm -> TerminalBlock_XINYA:TerminalBlock_XINYA_XY301-1x3-P5.00mm
- renumbered J3 to J4, J4 to J6, J5 to J8
Connections:
- net +12V: now also J3.10 (Pin_10), J3.9 (Pin_9), J5.10 (Pin_10), J5.9 (Pin_9), J9.10 (Pin_10), J9.9 (Pin_9)
- net -12V: now also J3.1 (Pin_1), J3.2 (Pin_2), J5.1 (Pin_1), J5.2 (Pin_2), J9.1 (Pin_1), J9.2 (Pin_2)
- net GND: now also J3.3 (Pin_3), J3.4 (Pin_4), J3.5 (Pin_5), J3.6 (Pin_6), J3.7 (Pin_7), J3.8 (Pin_8), J5.3 (Pin_3), J5.4 (Pin_4), J5.5 (Pin_5), J5.6 (Pin_6), J5.7 (Pin_7), J5.8 (Pin_8), J9.3 (Pin_3), J9.4 (Pin_4), J9.5 (Pin_5), J9.6 (Pin_6), J9.7 (Pin_7), J9.8 (Pin_8)
Other:
- moved on the sheet: J1, J10, J2, J4, J6, J8
